Commit message: changed box size

File: robots/box.xacro (robot description, xacro)
@@ -18,5 +18,5 @@
             <origin xyz="0 0 0"/>
             <geometry>
-                <box size="0.02 0.02 1.99" />
+                <box size="0.02 0.02 0.2" />
             </geometry>
         </visual>
@@ -24,5 +24,5 @@
             <origin xyz="0 0 0"/>
             <geometry>
-                <box size="0.02 0.02 1.99" />
+                <box size="0.02 0.02 0.2" />
             </geometry>
         </collision>

Commit message: changed box sizes

File: robots/box.xacro (robot description, xacro)
@@ -18,5 +18,5 @@
             <origin xyz="0 0 0"/>
             <geometry>
-                <box size="0.02 0.02 0.2" />
+                <box size="0.025 0.025 0.2" />
             </geometry>
         </visual>
@@ -24,5 +24,5 @@
             <origin xyz="0 0 0"/>
             <geometry>
-                <box size="0.02 0.02 0.2" />
+                <box size="0.025 0.025 0.2" />
             </geometry>
         </collision>
